File: hw/through-hole/0.2.0/CO2 Monitor Through Hole.kicad_pcb (KiCad board)
At the start: 2 copper layers, 81.3 x 80.8 mm, 27 parts

Commit message: minor silkscreen updates
Parts:
- REF** (x3): moved to F.Cu
- moved REF** 34.1 mm to (96.8, 93.5), turned to 0 degrees
- moved REF** 14.5 mm to (75.9, 88.1), turned to 0 degrees
- moved REF** 14.0 mm to (85.6, 93.7), turned to 0 degrees
- moved G*** 7.15 mm to (89.5, 88.1)
