File: hw/through-hole/0.2.1-old/CO2 Monitor Through Hole.kicad_pcb (KiCad board)
At the start: 2 copper layers, 82 x 90 mm, 29 parts

Commit message: updated 0.2.1 hardware
added software tests
Parts:
- moved H2 0.51 mm to (125.7, 43.9)
- moved H4 0.51 mm to (125.7, 118.4)
Other:
- board size 82 x 90 mm -> 81.3 x 80.8 mm
Changed lines of the file:
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@@
 			(plot_on_all_layers_selection 0x0000000_00000000)
 			(disableapertmacros no)
-			(usegerberextensions yes)
-			(usegerberattributes no)
-			(usegerberadvancedattributes no)
-			(creategerberjobfile no)
+			(usegerberextensions no)
+			(usegerberattributes yes)
+			(usegerberadvancedattributes yes)
+			(creategerberjobfile yes)
 			(dashed_line_dash_ratio 12.000000)
 			(dashed_line_gap_ratio 3.000000)
@@
 			(psa4output no)
 			(plotreference yes)
-			(plotvalue no)
+			(plotvalue yes)
 			(plotfptext yes)
 			(plotinvisibletext no)
 			(sketchpadsonfab no)
-			(subtractmaskfromsilk yes)
+			(subtractmaskfromsilk no)
 			(outputformat 1)
 			(mirror no)
-			(drillshape 0)
+			(drillshape 1)
 			(scaleselection 1)
-			(outputdirectory "plots/")
+			(outputdirectory "")
 		)
 	)
@@
 			)
 		)
-		(model "/Users/romkey/Downloads/SM04B-SRSS-TB.STEP"
-			(offset
-				(xyz 0 1.5 0)
-			)
-			(scale
-				(xyz 1 1 1)
-			)
-			(rotate
-				(xyz -90 0 0)
-			)
-		)
 	)
 	(footprint "1myFootprints:Adafruit eInk Breakout Friend"
@@
 	(footprint "MountingHole:MountingHole_2.7mm_M2.5"
 		(layer "F.Cu")
-		(at 126.238 118.364)
+		(at 125.73 118.364)
 		(descr "Mounting Hole 2.7mm, no annular, M2.5")
 		(tags "mounting hole 2.7mm no annular m2.5")
@@
 			(layer "F.Fab")
 		)
-		(fp_text user "RX"
-			(at -1.25 -9.0365 -90)
+		(fp_text user "PMS5003"
+			(at 7.783 -9.7985 0)
 			(unlocked yes)
 			(layer "F.SilkS")
@@
 					(thickness 0.1)
 				)
-				(justify left)
+				(justify left bottom)
 			)
 		)
-		(fp_text user "TX"
-			(at 0.5 -9.0365 -90)
+		(fp_text user "VCC"
+			(at -4.98 -9.0365 -90)
 			(unlocked yes)
 			(layer "F.SilkS")
@@
 					(thickness 0.1)
 				)
-				(justify left bottom)
+				(justify left)
 			)
 		)
-		(fp_text user "RESET"
-			(at 1.5 -9.0365 -90)
+		(fp_text user "SET"
+			(at -2.5 -9.0365 -90)
 			(unlocked yes)
 			(layer "F.SilkS")
@@
 			)
 		)
-		(fp_text user "VCC"
-			(at -4.98 -9.0365 -90)
+		(fp_text user "RX"
+			(at -1.25 -9.0365 -90)
 			(unlocked yes)
 			(layer "F.SilkS")
@@
 			)
 		)
-		(fp_text user "SET"
-			(at -2.5 -9.0365 -90)
+		(fp_text user "TX"
+			(at 0.5 -9.0365 -90)
 			(unlocked yes)
 			(layer "F.SilkS")
@@
 					(thickness 0.1)
 				)
-				(justify left)
+				(justify left bottom)
 			)
 		)
-		(fp_text user "PMS5003"
-			(at 7.783 -9.7985 0)
+		(fp_text user "RESET"
+			(at 1.5 -9.0365 -90)
 			(unlocked yes)
 			(layer "F.SilkS")
@@
 					(thickness 0.1)
 				)
-				(justify left bottom)
-			)
-		)
-		(fp_text user "${REFERENCE}"
-			(at 0 2.5 180)
-			(unlocked yes)
-			(layer "F.Fab")
-			(effects
-				(font
-					(size 1 1)
-					(thickness 0.15)
-				)
+				(justify left)
 			)
 		)
@@
 			(solder_mask_margin 0.0762)
 		)
-		(model "/Users/romkey/Downloads/0532610871/53261-0871.step"
-			(opacity 0.8000)
-			(offset
-				(xyz -0.5 3.5 1.7)
-			)
-			(scale
-				(xyz 1 1 1)
-			)
-			(rotate
-				(xyz 180 180 0)
-			)
-		)
 	)
 	(footprint "1myFootprints:SPI_TFT_TOUCH"
@@
 	(footprint "MountingHole:MountingHole_2.7mm_M2.5"
 		(layer "F.Cu")
-		(at 126.238 43.942)
+		(at 125.73 43.942)
 		(descr "Mounting Hole 2.7mm, no annular, M2.5")
 		(tags "mounting hole 2.7mm no annular m2.5")
@@
 	)
 	(gr_rect
-		(start 47.392 31.666)
-		(end 129.392 121.666)
-		(stroke
-			(width 0.1)
-			(type default)
-		)
-		(fill none)
-		(layer "Edge.Cuts")
-	)
-	(gr_rect
-		(start 79.404 33.298)
-		(end 87.404 36.298)
-		(stroke
-			(width 0.1)
-			(type default)
-		)
-		(fill none)
-		(layer "Edge.Cuts")
-	)
-	(gr_rect
-		(start 49.404 33.298)
-		(end 57.404 36.298)
-		(stroke
-			(width 0.1)
-			(type default)
-		)
-		(fill none)
-		(layer "Edge.Cuts")
-	)
-	(gr_rect
-		(start 89.404 33.298)
-		(end 97.404 36.298)
-		(stroke
-			(width 0.1)
-			(type default)
-		)
-		(fill none)
-		(layer "Edge.Cuts")
-	)
-	(gr_rect
-		(start 69.404 33.298)
-		(end 77.404 36.298)
-		(stroke
-			(width 0.1)
-			(type default)
-		)
-		(fill none)
-		(layer "Edge.Cuts")
-	)
-	(gr_rect
-		(start 59.404 33.298)
-		(end 67.404 36.298)
+		(start 47.498 40.64)
+		(end 128.778 121.412)
 		(stroke
 			(width 0.1)
@@
 		(stroke
 			(width 0.1)
-			(type default)
-		)
-		(fill none)
-		(layer "Edge.Cuts")
-	)
-	(gr_rect
-		(start 109.404 33.298)
-		(end 117.404 36.298)
-		(stroke
-			(width 0.1)
-			(type default)
-		)
-		(fill none)
-		(layer "Edge.Cuts")
-	)
-	(gr_rect
-		(start 119.404 33.298)
-		(end 127.404 36.298)
-		(stroke
-			(width 0.1)
-			(type default)
-		)
-		(fill none)
-		(layer "Edge.Cuts")
-	)
-	(gr_rect
-		(start 99.404 33.298)
-		(end 107.404 36.298)
-		(stroke
-			(width 0.1)
