File: hw/through-hole/0.2.1-old/CO2 Monitor Through Hole.kicad_sch (KiCad schematic)
At the start: 25 parts

Commit message: updated 0.2.1 hardware
added software tests
Parts:
- U1: footprint 1myFootprints:Xiao ESP32S3 Sense (Camera) -> 1myFootprints:Xiao ESP32S3
Changed lines of the file:
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@@
 			)
 		)
-		(property "Footprint" "1myFootprints:Xiao ESP32S3 Sense (Camera)"
+		(property "Footprint" "1myFootprints:Xiao ESP32S3"
 			(at 57.15 57.15 0)
 			(effects
